Commit message: Description: Developed a preeliminary urdf

File: g_mov_description/urdf/g_mov.urdf.xacro (robot description, xacro)
@@ -1,6 +1,9 @@
 <?xml version="1.0"?>
 <robot xmlns:xacro="http://www.ros.org/wiki/xacro" name="orion">
-   <!-- Include other files -->
+    <!-- Include other files -->
+    <xacro:include filename="$(find g_mov_description)/urdf/g_mov_materials.urdf.xacro"/>
     <xacro:include filename="$(find g_mov_description)/urdf/g_mov_macros.urdf.xacro"/>
     <link name="base_link"/>
+    <xacro:g_mov_assem parent="base_link" spacer="m3x10" offset="${0.033/2}"
+        x="0" y="0" z="0"/>
 </robot>

File: g_mov_description/urdf/g_mov_macros.urdf.xacro (robot description, xacro)
@@ -3,6 +3,6 @@
 <!--///////////////////// M3 x 10 SPACERS MACROS ///////////////////////-->
     <xacro:macro name="generic_spacer"
-            params="id parent element front side x y z m xx xy xz yy yz zz">
-        <!-- Link -->
+            params="id parent element front side x y z">
+        <!-- Link Spacer -->
         <link name="${id}_${element}_${front}${side}">
         <visual>
@@ -23,10 +23,25 @@
         <inertial>
             <origin xyz="0 0 0 " rpy="0 0 0"/>
-            <mass value="${m}"/>
-            <inertia ixx="${xx}" ixy="${xy}" ixz="${xz}"
-                    iyy="${yy}" iyz="${yz}"
-                    izz="${zz}"/>
-        </inertial>
-        </link>
+            <xacro:if value="${id == 'm3x20'}">
+                <mass value="0.0024"/>
+                <inertia ixx="8.5251996963501e-08" ixy="0" ixz="0"
+                        iyy="8.648216387229408e-08" iyz="0"
+                        izz="1.333016690879308e-08"/>
+            </xacro:if>
+            <xacro:if value="${id == 'm3x10'}">
+                <mass value="0.0012"/>
+                <inertia ixx="1.2825999244689955e-08" ixy="0" ixz="0"
+                        iyy="1.3441082699086494e-08" iyz="0"
+                        izz="6.66508345439654e-09"/>
+            </xacro:if>
+            <xacro:if value="${id == 'm3x6'}">
+                <mass value="0.00072"/>
+                <inertia ixx="3.9036000675201425e-09" ixy="0" ixz="0"
+                        iyy=".272650140158067e-09" iyz="0"
+                        izz="3.9990500726379235e-09"/>
+            </xacro:if>
+        </inertial>
+        </link>
+        <!-- Joint Spacer -->
         <joint name="${id}_${element}_${front}${side}_joint" type="fixed">
             <parent link="${parent}"/>
@@ -38,12 +53,247 @@
     <xacro:macro name="x4xgeneric_spacer"
                 params="id element parent offset_x offset_y x y z">
-        <xacro:spacer_m3x10 id="${id}" parent="${parent}" element="${element}"
+        <xacro:generic_spacer id="${id}" parent="${parent}" element="${element}"
             front="f" side="r" x="${x + offset_x}" y="${y - offset_y}" z="${z}"/>
-        <xacro:spacer_m3x10 id="${id}" parent="${parent}" element="${element}"
+        <xacro:generic_spacer id="${id}" parent="${parent}" element="${element}"
             front="f" side="l" x="${x + offset_x}" y="${y + offset_y}" z="${z}"/>
-        <xacro:spacer_m3x10 id="${id}" parent="${parent}" element="${element}"
+        <xacro:generic_spacer id="${id}" parent="${parent}" element="${element}"
             front="r" side="r" x="${x - offset_x}" y="${y + offset_y}" z="${z}"/>
-        <xacro:spacer_m3x10 id="${id}" parent="${parent}" element="${element}"
+        <xacro:generic_spacer id="${id}" parent="${parent}" element="${element}"
             front="r" side="l" x="${x - offset_x}" y="${y - offset_y}" z="${z}"/>
     </xacro:macro>
+    <xacro:macro name="g_mov_assem" params="parent spacer offset x y z">
+        <xacro:property name="heigh_level" value="0.005"/>
+        <xacro:if value="${spacer == 'm3x20'}">
+            <xacro:property name="heigh_level" value="0.020"/>
+        </xacro:if>
+        <xacro:if value="${spacer == 'm3x10'}">
+            <xacro:property name="heigh_level" value="0.010"/>
+        </xacro:if>
+        <xacro:if value="${spacer == 'm3x6'}">
+            <xacro:property name="heigh_level" value="0.006"/>
+        </xacro:if>
+        <xacro:x4xgeneric_spacer id="${spacer}" element="${parent}" parent="${parent}"
+            offset_x="${0.06365/2}" offset_y="${offset}" x="${x}" y="${y}" z="${z}"/>
+        <!-- Link Accel -->
+        <link name="accel_base">
+        <visual>
+            <origin xyz="0 0 0" rpy="0 0 0"/>
+            <geometry>
+            <mesh filename="package://g_mov_description/meshes/accel_base.stl"
+                scale="0.001 0.001 0.001"/>
+            </geometry>
+            <material name="PLAGray"/>
+        </visual>
+        <collision>
+            <origin xyz="0 0 0" rpy="0 0 0"/>
+            <geometry>
+            <mesh filename="package://g_mov_description/meshes/accel_base.stl"
+                scale="0.001 0.001 0.001"/>
+            </geometry>
+        </collision>
+        <inertial>
+            <origin xyz="0 0 0 " rpy="0 0 0"/>
+                <mass value="0.008"/>
+                <inertia ixx="1.1233333333333333e-06" ixy="0" ixz="0"
+                        iyy="3.458666666666666e-06" iyz="0"
+                        izz="4.576666666666666e-06"/>
+        </inertial>
+        </link>
+        <!-- Joint Accel Base -->
+        <joint name="accel_base_joint" type="fixed">
+            <parent link="${parent}"/>
+            <child link="accel_base"/>
+            <origin xyz="${x} ${y} ${z + heigh_level}" rpy="0 0 0"/>
+        </joint>
+        <!-- Link Accel -->
+        <link name="accel">
+        <visual>
+            <origin xyz="0 0 0" rpy="0 0 0"/>
+            <geometry>
+            <mesh filename="package://g_mov_description/meshes/accel.stl"
+                scale="0.001 0.001 0.001"/>
+            </geometry>
+            <material name="ArduinoBlue"/>
+        </visual>
+        <collision>
+            <origin xyz="0 0 0" rpy="0 0 0"/>
+            <geometry>
+            <mesh filename="package://g_mov_description/meshes/accel.stl"
+                scale="0.001 0.001 0.001"/>
+            </geometry>
+        </collision>
+        <inertial>
+            <origin xyz="0 0 0 " rpy="0 0 0"/>
+                <mass value="0.009"/>
+                <inertia ixx="4.064043630409241e-07" ixy="0" ixz="0"
+                        iyy="2.879643941116337e-07" iyz="0"
+                        izz="5.367750071525579e-07"/>
+        </inertial>
+        </link>
+        <!-- Joint Accel -->
+        <joint name="accel_joint" type="fixed">
+            <parent link="accel_base"/>
+            <child link="accel"/>
+            <origin xyz="0.00025 0 0.00175" rpy="0 0 0"/>
+        </joint>
+        <xacro:x4xgeneric_spacer id="${spacer}" element="accel_base" parent="accel_base"
+            offset_x="${0.06365/2}" offset_y="${offset}" x="0" y="0" z="0.00175"/>
+        <!-- Link servo_base -->
+        <link name="servo_base">
+        <visual>
+            <origin xyz="0 0 0" rpy="0 0 0"/>
+            <geometry>
+            <mesh filename="package://g_mov_description/meshes/servo_base.stl"
+                scale="0.001 0.001 0.001"/>
+            </geometry>
+            <material name="PLAGray"/>
+        </visual>
+        <collision>
+            <origin xyz="0 0 0" rpy="0 0 0"/>
+            <geometry>
+            <mesh filename="package://g_mov_description/meshes/servo_base.stl"
+                scale="0.001 0.001 0.001"/>
+            </geometry>
+        </collision>
+        <inertial>
+            <origin xyz="0 0 0 " rpy="0 0 0"/>
+                <mass value="0.012"/>
+                <inertia ixx="2.21e-06" ixy="0" ixz="0"
+                        iyy="5.713e-06" iyz="0"
+                        izz="6.8649999999999995e-06"/>
+        </inertial>
+        </link>
+        <!-- Joint servo base -->
+        <joint name="servo_base_joint" type="fixed">
+            <parent link="accel_base"/>
+            <child link="servo_base"/>
+            <origin xyz="0.00025 0 ${0.00175+heigh_level}" rpy="0 0 0"/>
+        </joint>
+        <!-- Link servo -->
+        <link name="servo">
+        <visual>
+            <origin xyz="0 0 0" rpy="${-pi/2} 0 0"/>
+            <geometry>
+            <mesh filename="package://g_mov_description/meshes/servo_mg996r.stl"
+                scale="0.001 0.001 0.001"/>
+            </geometry>
+            <material name="SoftBlack"/>
+        </visual>
+        <collision>
+            <origin xyz="0 0 0" rpy="${-pi/2} 0 0"/>
+            <geometry>
+            <mesh filename="package://g_mov_description/meshes/servo_mg996r.stl"
+                scale="0.001 0.001 0.001"/>
+            </geometry>
+        </collision>
+        <inertial>
+            <origin xyz="0 0 0 " rpy="${pi/2} 0 0"/>
+                <mass value="0.055"/>
+                <inertia ixx="1.1155878535842904e-05" ixy="0" ixz="0"
+                        iyy="2.1057527828089415e-05" iyz="0"
+                        izz="1.3568315958913178e-05"/>
+        </inertial>
+        </link>
+        <!-- Joint servo -->
+        <joint name="servo_joint" type="fixed">
+            <parent link="servo_base"/>
+            <child link="servo"/>
+            <origin xyz="0 -0.0185 ${0.00175 + 0.01}" rpy="0 0 0"/>
+        </joint>
+        <!-- Link servo conn -->
+        <link name="servo_conn">
+        <visual>
+            <origin xyz="0 0 0" rpy="0 0 0"/>
+            <geometry>
+            <mesh filename="package://g_mov_description/meshes/servo_conn.stl"
+                scale="0.001 0.001 0.001"/>
+            </geometry>
+            <material name="MetalGray"/>
+        </visual>
+        <collision>
+            <origin xyz="0 0 0" rpy="0 0 0"/>
+            <geometry>
+            <mesh filename="package://g_mov_description/meshes/servo_conn.stl"
+                scale="0.001 0.001 0.001"/>
+            </geometry>
+        </collision>
+        <inertial>
+            <origin xyz="0 0 0 " rpy="0 0 0"/>
+                <mass value="0.0024"/>
+                <inertia ixx="8.40345435933159e-08" ixy="0" ixz="0"
+                        iyy="8.401908867990422e-08" iyz="0"
+                        izz="1.5995363227322013e-07"/>
+        </inertial>
+        </link>
+        <!-- Joint servo conn -->
+        <joint name="servo_conn_joint" type="revolute">
+            <parent link="servo"/>
+            <child link="servo_conn"/>
+            <limit lower="${-pi/4}" upper="${pi/6}" effort="1.0" velocity="1.0"/>
+            <axis xyz="0.0 0.0 1.0"/>
+            <origin xyz="0.01 0.042 0" rpy="${-pi/2} 0 0"/>
+        </joint>
+        <!-- Link Pi Cam Support -->
+        <link name="picam_sup">
+        <visual>
+            <origin xyz="0 0 0" rpy="0 ${-pi/2} ${pi/2}"/>
+            <geometry>
+            <mesh filename="package://g_mov_description/meshes/picam_sup.stl"
+                scale="0.001 0.001 0.001"/>
+            </geometry>
+            <material name="PLAGray"/>
+        </visual>
+        <collision>
+            <origin xyz="0 0 0" rpy="0 ${-pi/2} ${pi/2}"/>
+            <geometry>
+            <mesh filename="package://g_mov_description/meshes/picam_sup.stl"
+                scale="0.001 0.001 0.001"/>
+            </geometry>
+        </collision>
+        <inertial>
+            <origin xyz="0 0 0 " rpy="0 ${-pi/2} ${pi/2}"/>
+                <mass value="0.008"/>
+                <inertia ixx="2.2308333333333333e-06" ixy="0" ixz="0"
+                        iyy="1.5268333333333331e-06" iyz="0"
+                        izz="3.1123333333333332e-06"/>
+        </inertial>
+        </link>
+        <!-- Joint Pi Cam Support -->
+        <joint name="picam_sup_joint" type="fixed">
+            <parent link="servo_conn"/>
+            <child link="picam_sup"/>
+            <origin xyz="0 0 0.005" rpy="0 0 0"/>
+        </joint>
+        <!-- Link Pi Cam -->
+        <link name="picam">
+        <visual>
+            <origin xyz="0 0 0" rpy="0 ${pi/2} 0"/>
+            <geometry>
+            <mesh filename="package://g_mov_description/meshes/picam.stl"
+                scale="0.001 0.001 0.001"/>
+            </geometry>
+            <material name="RaspberryGreen"/>
+        </visual>
+        <collision>
+            <origin xyz="0 0 0" rpy="0 ${pi/2} 0"/>
+            <geometry>
+            <mesh filename="package://g_mov_description/meshes/picam.stl"
+                scale="0.001 0.001 0.001"/>
+            </geometry>
+        </collision>
+        <inertial>
+            <origin xyz="0 0 0 " rpy="0 ${pi/2} 0"/>
+                <mass value="0.008"/>
+                <inertia ixx="2.2308333333333333e-06" ixy="0" ixz="0"
+                        iyy="1.5268333333333331e-06" iyz="0"
+                        izz="3.1123333333333332e-06"/>
+        </inertial>
+        </link>
+        <!-- Joint Pi Cam -->
+        <joint name="picam_joint" type="fixed">
+            <parent link="picam_sup"/>
+            <child link="picam"/>
+            <origin xyz="0.038 -0.004 -0.0275" rpy="0 0 0"/>
+        </joint>
+    </xacro:macro>
 </robot>

Commit message: Description: Adding camera links and optical links

File: g_mov_description/urdf/g_mov.urdf.xacro (robot description, xacro)
@@ -6,4 +6,4 @@
     <link name="base_link"/>
     <xacro:g_mov_assem parent="base_link" spacer="m3x10" offset="${0.033/2}"
-        x="0" y="0" z="0"/>
+        x="0" y="0" z="0" joint_prefix="g_mov"/>
 </robot>

File: g_mov_description/urdf/g_mov_macros.urdf.xacro (robot description, xacro)
@@ -1,8 +1,8 @@
 <?xml version="1.0"?>
 <robot xmlns:xacro="http://www.ros.org/wiki/xacro">
-<!--///////////////////// M3 x 10 SPACERS MACROS ///////////////////////-->
+    <!--///////////////////// GENERIC SPACERS MACROS ///////////////////////-->
+    <!-- ...................... Single spacers ............................ -->
     <xacro:macro name="generic_spacer"
             params="id parent element front side x y z">
-        <!-- Link Spacer -->
         <link name="${id}_${element}_${front}${side}">
         <visual>
@@ -43,5 +43,4 @@
         </inertial>
         </link>
-        <!-- Joint Spacer -->
         <joint name="${id}_${element}_${front}${side}_joint" type="fixed">
             <parent link="${parent}"/>
@@ -62,5 +61,23 @@
             front="r" side="l" x="${x - offset_x}" y="${y - offset_y}" z="${z}"/>
     </xacro:macro>
-    <xacro:macro name="g_mov_assem" params="parent spacer offset x y z">
+    <!-- /////////////////////// Sensors macros ////////////////////////// -->
+    <xacro:macro name="add_cam_links" params="x y z R P Y parent">
+        <!-- ................... Camera sensors links .................. -->
+        <link name="g_mov_cam_link"/>
+        <joint name="g_mov_cam_joint" type="fixed">
+            <origin xyz="${x} ${y} ${z}" rpy="0 0 0"/>
+            <parent link="${parent}"/>
+            <child link="g_mov_cam_link"/>
+        </joint>
+        <link name="g_mov_cam_link_optical"/>
+        <joint name="g_mov_optical_joint" type="fixed">
+            <origin xyz="0 0 0" rpy="${R} ${P} ${Y}"/>
+            <parent link="g_mov_cam_link"/>
+            <child link="g_mov_cam_link_optical"/>
+        </joint>
+    </xacro:macro>
+    <!-- //////////////////////////// Assemblys macros ////////////////////////// -->
+    <xacro:macro name="g_mov_assem" params="parent spacer offset x y z joint_prefix">
+        <!-- Properties -->
         <xacro:property name="heigh_level" value="0.005"/>
         <xacro:if value="${spacer == 'm3x20'}">
@@ -73,4 +90,5 @@
             <xacro:property name="heigh_level" value="0.006"/>
         </xacro:if>
+        <!-- Spacers -->
         <xacro:x4xgeneric_spacer id="${spacer}" element="${parent}" parent="${parent}"
             offset_x="${0.06365/2}" offset_y="${offset}" x="${x}" y="${y}" z="${z}"/>
@@ -100,5 +118,4 @@
         </inertial>
         </link>
-        <!-- Joint Accel Base -->
         <joint name="accel_base_joint" type="fixed">
             <parent link="${parent}"/>
@@ -131,5 +148,4 @@
         </inertial>
         </link>
-        <!-- Joint Accel -->
         <joint name="accel_joint" type="fixed">
             <parent link="accel_base"/>
@@ -137,4 +153,5 @@
             <origin xyz="0.00025 0 0.00175" rpy="0 0 0"/>
         </joint>
+        <!-- Spacers -->
         <xacro:x4xgeneric_spacer id="${spacer}" element="accel_base" parent="accel_base"
             offset_x="${0.06365/2}" offset_y="${offset}" x="0" y="0" z="0.00175"/>
@@ -164,5 +181,4 @@
         </inertial>
         </link>
-        <!-- Joint servo base -->
         <joint name="servo_base_joint" type="fixed">
             <parent link="accel_base"/>
@@ -195,5 +211,4 @@
         </inertial>
         </link>
-        <!-- Joint servo -->
         <joint name="servo_joint" type="fixed">
             <parent link="servo_base"/>
@@ -226,6 +241,5 @@
         </inertial>
         </link>
-        <!-- Joint servo conn -->
-        <joint name="servo_conn_joint" type="revolute">
+        <joint name="${joint_prefix}_servo_conn_joint" type="revolute">
             <parent link="servo"/>
             <child link="servo_conn"/>
@@ -259,5 +273,4 @@
         </inertial>
         </link>
-        <!-- Joint Pi Cam Support -->
         <joint name="picam_sup_joint" type="fixed">
             <parent link="servo_conn"/>
@@ -290,5 +303,4 @@
         </inertial>
         </link>
-        <!-- Joint Pi Cam -->
         <joint name="picam_joint" type="fixed">
             <parent link="picam_sup"/>
@@ -296,4 +308,7 @@
             <origin xyz="0.038 -0.004 -0.0275" rpy="0 0 0"/>
         </joint>
+        <!-- Camera reference -->
+        <xacro:add_cam_links x="0.0065" y="-0.003" z="0" R="0" P="${pi/2}" Y="0"
+          parent="picam"/>
     </xacro:macro>
 </robot>
