Commit message: Description: Adding Gazebo control and camera

File: g_mov_description/urdf/g_mov.urdf.xacro (robot description, xacro)
@@ -1,4 +1,5 @@
 <?xml version="1.0"?>
 <robot xmlns:xacro="http://www.ros.org/wiki/xacro" name="orion">
+    <xacro:property name="gazebo" value="false"/>
     <!-- Include other files -->
     <xacro:include filename="$(find g_mov_description)/urdf/g_mov_materials.urdf.xacro"/>

File: g_mov_description/urdf/g_mov_macros.urdf.xacro (robot description, xacro)
@@ -48,4 +48,10 @@
             <origin xyz="${x} ${y} ${z}" rpy="0 0 0"/>
         </joint>
+        <xacro:if value="${gazebo}">
+            <gazebo reference="${id}_${element}_${front}${side}">
+                <mu1>1.0</mu1>
+                <mu2>1.0</mu2>
+            </gazebo>
+        </xacro:if>
     </xacro:macro>
     <!-- 4 symetric hex spacers by considering x/y axis -->
@@ -66,5 +72,5 @@
         <link name="g_mov_cam_link"/>
         <joint name="g_mov_cam_joint" type="fixed">
-            <origin xyz="${x} ${y} ${z}" rpy="0 0 0"/>
+            <origin xyz="${x} ${y} ${z}" rpy="${-pi/2} 0 0"/>
             <parent link="${parent}"/>
             <child link="g_mov_cam_link"/>
@@ -123,4 +129,10 @@
             <origin xyz="${x} ${y} ${z + heigh_level}" rpy="0 0 0"/>
         </joint>
+        <xacro:if value="${gazebo}">
+            <gazebo reference="accel_base">
+                <mu1>1.0</mu1>
+                <mu2>1.0</mu2>
+            </gazebo>
+        </xacro:if>
         <!-- Link Accel -->
         <link name="accel">
@@ -153,4 +165,10 @@
             <origin xyz="0.00025 0 0.00175" rpy="0 0 0"/>
         </joint>
+        <xacro:if value="${gazebo}">
+            <gazebo reference="accel">
+                <mu1>1.0</mu1>
+                <mu2>1.0</mu2>
+            </gazebo>
+        </xacro:if>
         <!-- Spacers -->
         <xacro:x4xgeneric_spacer id="${spacer}" element="accel_base" parent="accel_base"
@@ -186,4 +204,10 @@
             <origin xyz="0.00025 0 ${0.00175+heigh_level}" rpy="0 0 0"/>
         </joint>
+        <xacro:if value="${gazebo}">
+            <gazebo reference="servo_base">
+                <mu1>1.0</mu1>
+                <mu2>1.0</mu2>
+            </gazebo>
+        </xacro:if>
         <!-- Link servo -->
         <link name="servo">
@@ -216,4 +240,10 @@
             <origin xyz="0 -0.0185 ${0.00175 + 0.01}" rpy="0 0 0"/>
         </joint>
+        <xacro:if value="${gazebo}">
+            <gazebo reference="servo">
+                <mu1>1.0</mu1>
+                <mu2>1.0</mu2>
+            </gazebo>
+        </xacro:if>
         <!-- Link servo conn -->
         <link name="servo_conn">
@@ -248,4 +278,25 @@
             <origin xyz="0.01 0.042 0" rpy="${-pi/2} 0 0"/>
         </joint>
+        <xacro:if value="${gazebo}">
+        <gazebo>
+            <plugin
+                filename="gz-sim-joint-position-controller-system"
+                name="gz::sim::systems::JointPositionController">
+                <joint_name>${joint_prefix}_servo_conn_joint</joint_name>
+                <topic>g_mov_servo</topic>
+                <p_gain>1</p_gain>
+                <i_gain>0.1</i_gain>
+                <d_gain>0.01</d_gain>
+                <i_max>1</i_max>
+                <i_min>-1</i_min>
+                <cmd_max>1000</cmd_max>
+                <cmd_min>-1000</cmd_min>
+            </plugin>
+        </gazebo>
+            <gazebo reference="servo_conn">
+                <mu1>1.0</mu1>
+                <mu2>1.0</mu2>
+            </gazebo>
+        </xacro:if>
         <!-- Link Pi Cam Support -->
         <link name="picam_sup">
@@ -278,4 +329,10 @@
             <origin xyz="0 0 0.005" rpy="0 0 0"/>
         </joint>
+        <xacro:if value="${gazebo}">
+            <gazebo reference="picam_sup">
+                <mu1>1.0</mu1>
+                <mu2>1.0</mu2>
+            </gazebo>
+        </xacro:if>
         <!-- Link Pi Cam -->
         <link name="picam">
@@ -308,7 +365,53 @@
             <origin xyz="0.038 -0.004 -0.0275" rpy="0 0 0"/>
         </joint>
+        <xacro:if value="${gazebo}">
+            <gazebo reference="picam_sup">
+                <mu1>1.0</mu1>
+                <mu2>1.0</mu2>
+            </gazebo>
+        </xacro:if>
         <!-- Camera reference -->
         <xacro:add_cam_links x="0.0065" y="-0.003" z="0" R="0" P="${pi/2}" Y="0"
           parent="picam"/>
+        <xacro:if value="${gazebo}">
+            <gazebo reference="g_mov_cam_link">
+                <sensor name="camera" type="camera">
+                    <!-- Data based on : -->
+                    <!-- https://static.chipdip.ru/lib/664/DOC001664108.pdf -->
+                    <camera>
+                        <horizontal_fov>1.361357</horizontal_fov>
+                        <image>
+                        <width>1080</width>
+                        <height>810</height>
+                        </image>
+                        <clip>
+                            <near>0.2</near>
+                            <far>10.0</far>
+                        </clip>
+                        <xacro:if value="true">
+                            <!-- Noise addition -->
+                            <noise>
+                                <type>gaussian</type>
+                                <mean>0.0</mean>
+                                <stddev>0.015</stddev>
+                            </noise>
+                            <!-- Distorsion addition -->
+                            <distortion>
+                                <k1>-0.1</k1>
+                                <k2>0.02</k2>
+                                <k3>0.01</k3>
+                                <p1>0.0</p1>
+                                <p2>0.0</p2>
+                                <center>0.5 0.5</center>
+                            </distortion>
+                        </xacro:if>
+                    </camera>
+                    <always_on>1</always_on>
+                    <update_rate>30</update_rate>
+                    <visualize>true</visualize>
+                    <topic>pi_cam</topic>
+                </sensor>
+            </gazebo>
+        </xacro:if>
     </xacro:macro>
 </robot>

Commit message: Description: Divide sensors to another xacro file | Gazebo: Added spawn module and basic ros_gz bridge

File: g_mov_description/urdf/g_mov.urdf.xacro (robot description, xacro)
@@ -1,8 +1,11 @@
 <?xml version="1.0"?>
 <robot xmlns:xacro="http://www.ros.org/wiki/xacro" name="orion">
-    <xacro:property name="gazebo" value="false"/>
+    <xacro:property name="gazebo" value="$(arg gazebo)"/>
     <!-- Include other files -->
     <xacro:include filename="$(find g_mov_description)/urdf/g_mov_materials.urdf.xacro"/>
     <xacro:include filename="$(find g_mov_description)/urdf/g_mov_macros.urdf.xacro"/>
+    <xacro:if value="${gazebo}">
+        <xacro:include filename="$(find g_mov_description)/urdf/g_mov_gz.urdf.xacro"/>
+    </xacro:if>
     <link name="base_link"/>
     <xacro:g_mov_assem parent="base_link" spacer="m3x10" offset="${0.033/2}"

File: g_mov_description/urdf/g_mov_macros.urdf.xacro (robot description, xacro)
@@ -177,91 +177,4 @@
             <child link="imu"/>
         </joint>
-        <xacro:if value="${gazebo}">
-            <gazebo>
-                <plugin
-                    filename="gz-sim-imu-system"
-                    name="gz::sim::systems::Imu">
-                </plugin>
-            </gazebo>
-            <gazebo reference="imu">
-                <sensor name="imu_sensor" type="imu">
-                    <always_on>1</always_on>
-                    <update_rate>50</update_rate>
-                    <imu>
-                    <enable_orientation>true</enable_orientation>
-                    <angular_velocity>
-                        <x>
-                        <noise type="gaussian">
-                            <mean>0</mean>
-                            <stddev>0.009</stddev>
-                            <bias_mean>0.00075</bias_mean>
-                            <bias_stddev>0.005</bias_stddev>
-                            <dynamic_bias_stddev>0.00002</dynamic_bias_stddev>
-                            <dynamic_bias_correlation_time>400.0</dynamic_bias_correlation_time>
-                            <precision>0.00025</precision>
-                        </noise>
-                        </x>
-                        <y>
-                        <noise type="gaussian">
-                            <mean>0</mean>
-                            <stddev>0.009</stddev>
-                            <bias_mean>0.00075</bias_mean>
-                            <bias_stddev>0.005</bias_stddev>
-                            <dynamic_bias_stddev>0.00002</dynamic_bias_stddev>
-                            <dynamic_bias_correlation_time>400.0</dynamic_bias_correlation_time>
-                            <precision>0.00025</precision>
-                        </noise>
-                        </y>
-                        <z>
-                        <noise type="gaussian">
-                            <mean>0</mean>
-                            <stddev>0.009</stddev>
-                            <bias_mean>0.00075</bias_mean>
-                            <bias_stddev>0.005</bias_stddev>
-                            <dynamic_bias_stddev>0.00002</dynamic_bias_stddev>
-                            <dynamic_bias_correlation_time>400.0</dynamic_bias_correlation_time>
-                            <precision>0.00025</precision>
-                        </noise>
-                        </z>
-                    </angular_velocity>
-                    <linear_acceleration>
-                        <x>
-                        <noise type="gaussian">
-                            <mean>0</mean>
-                            <stddev>0.021</stddev>
-                            <bias_mean>0.05</bias_mean>
-                            <bias_stddev>0.0075</bias_stddev>
-                            <dynamic_bias_stddev>0.000375</dynamic_bias_stddev>
-                            <dynamic_bias_correlation_time>175.0</dynamic_bias_correlation_time>
-                            <precision>0.005</precision>
-                        </noise>
-                        </x>
-                        <y>
-                        <noise type="gaussian">
-                            <mean>0</mean>
-                            <stddev>0.021</stddev>
-                            <bias_mean>0.05</bias_mean>
-                            <bias_stddev>0.0075</bias_stddev>
-                            <dynamic_bias_stddev>0.000375</dynamic_bias_stddev>
-                            <dynamic_bias_correlation_time>175.0</dynamic_bias_correlation_time>
-                            <precision>0.005</precision>
-                        </noise>
-                        </y>
-                        <z>
-                        <noise type="gaussian">
-                            <mean>0</mean>
-                            <stddev>0.021</stddev>
-                            <bias_mean>0.05</bias_mean>
-                            <bias_stddev>0.0075</bias_stddev>
-                            <dynamic_bias_stddev>0.000375</dynamic_bias_stddev>
-                            <dynamic_bias_correlation_time>175.0</dynamic_bias_correlation_time>
-                            <precision>0.005</precision>
-                        </noise>
-                        </z>
-                    </linear_acceleration>
-                    </imu>
-                </sensor>
-            </gazebo>
-        </xacro:if>
         <!-- Spacers -->
         <xacro:x4xgeneric_spacer id="${spacer}" element="accel_base" parent="accel_base"
@@ -367,5 +280,6 @@
             <parent link="servo"/>
             <child link="servo_conn"/>
-            <limit lower="${-pi/4}" upper="${pi/6}" effort="1.0" velocity="1.0"/>
+            <limit lower="${-pi/4}" upper="${pi/6}" effort="0.92" velocity="6.0"/>
+            <dynamics damping="0.05" friction="0.02"/>
             <axis xyz="0.0 0.0 1.0"/>
             <origin xyz="0.01 0.042 0" rpy="${-pi/2} 0 0"/>
@@ -452,43 +366,4 @@
         <xacro:add_cam_links x="0.0065" y="-0.003" z="0" R="0" P="${pi/2}" Y="0"
           parent="picam"/>
-        <xacro:if value="${gazebo}">
-            <gazebo reference="g_mov_cam_link">
-                <sensor name="camera" type="camera">
-                    <!-- Data based on : -->
-                    <!-- https://static.chipdip.ru/lib/664/DOC001664108.pdf -->
-                    <camera>
-                        <horizontal_fov>1.361357</horizontal_fov>
-                        <image>
-                        <width>1080</width>
-                        <height>810</height>
-                        </image>
-                        <clip>
-                            <near>0.2</near>
-                            <far>10.0</far>
-                        </clip>
-                        <xacro:if value="true">
-                            <!-- Noise addition -->
-                            <noise>
-                                <type>gaussian</type>
-                                <mean>0.0</mean>
-                                <stddev>0.015</stddev>
-                            </noise>
-                            <!-- Distorsion addition -->
-                            <distortion>
-                                <k1>-0.1</k1>
-                                <k2>0.02</k2>
-                                <k3>0.01</k3>
-                                <p1>0.0</p1>
-                                <p2>0.0</p2>
-                                <center>0.5 0.5</center>
-                            </distortion>
-                        </xacro:if>
-                    </camera>
-                    <always_on>1</always_on>
-                    <update_rate>30</update_rate>
-                    <visualize>true</visualize>
-                </sensor>
-            </gazebo>
-        </xacro:if>
     </xacro:macro>
 </robot>

Commit message: Assets: Fixed on screw pockets and added fillets | Description: Updated URDF according new meshes

File: g_mov_description/urdf/g_mov.urdf.xacro (robot description, xacro)
@@ -9,5 +9,5 @@
     </xacro:if>
     <link name="base_link"/>
-    <xacro:g_mov_assem parent="base_link" spacer="m3x10" offset="${0.033/2}"
+    <xacro:g_mov_assem parent="base_link" spacer="m3x20" offset="${0.033/2}"
         x="0" y="0" z="0" joint_prefix="g_mov"/>
 </robot>

File: g_mov_description/urdf/g_mov_macros.urdf.xacro (robot description, xacro)
@@ -28,4 +28,10 @@
                         iyy="8.648216387229408e-08" iyz="0"
                         izz="1.333016690879308e-08"/>
+            </xacro:if>
+            <xacro:if value="${id == 'm3x15'}">
+                <mass value="0.0017"/>
+                <inertia ixx="5.2825999244689955e-08" ixy="0" ixz="0"
+                        iyy="5.4441082699086494e-08" iyz="0"
+                        izz="9.66508345439654e-09"/>
             </xacro:if>
             <xacro:if value="${id == 'm3x10'}">
@@ -72,5 +78,5 @@
         <link name="g_mov_cam_link"/>
         <joint name="g_mov_cam_joint" type="fixed">
-            <origin xyz="${x} ${y} ${z}" rpy="${-pi/2} 0 0"/>
+            <origin xyz="${x} ${y} ${z}" rpy="0 0 0"/>
             <parent link="${parent}"/>
             <child link="g_mov_cam_link"/>
@@ -90,4 +96,7 @@
             <xacro:property name="heigh_level" value="0.020"/>
         </xacro:if>
+        <xacro:if value="${spacer == 'm3x15'}">
+            <xacro:property name="heigh_level" value="0.015"/>
+        </xacro:if>
         <xacro:if value="${spacer == 'm3x10'}">
             <xacro:property name="heigh_level" value="0.010"/>
@@ -244,5 +253,5 @@
             <parent link="servo_base"/>
             <child link="servo"/>
-            <origin xyz="0 -0.0185 ${0.00175 + 0.01}" rpy="0 0 0"/>
+            <origin xyz="0 -0.01625 ${0.00175 + 0.01}" rpy="0 0 0"/>
         </joint>
         <xacro:if value="${gazebo}">
@@ -355,8 +364,8 @@
             <parent link="picam_sup"/>
             <child link="picam"/>
-            <origin xyz="0.038 -0.004 -0.0275" rpy="0 0 0"/>
-        </joint>
-        <xacro:if value="${gazebo}">
-            <gazebo reference="picam_sup">
+            <origin xyz="0.038 -0.004 -0.0275" rpy="${pi/2} 0 0"/>
+        </joint>
+        <xacro:if value="${gazebo}">
+            <gazebo reference="picam">
                 <mu1>1.0</mu1>
                 <mu2>1.0</mu2>
@@ -364,5 +373,5 @@
         </xacro:if>
         <!-- Camera reference -->
-        <xacro:add_cam_links x="0.0065" y="-0.003" z="0" R="0" P="${pi/2}" Y="0"
+        <xacro:add_cam_links x="0.0065" y="-0.003" z="0" R="${-pi/2}" P="0" Y="${-pi/2}"
           parent="picam"/>
     </xacro:macro>
